File: thermistor-measurement-board/bias-mux.sch (KiCad schematic (older format))
At the start: 28 parts, among them P201 BIAS, U201 MAX14661, U202 AD8607, U203 AD8277, U204 MAX6070, U205 MAX6070

Commit message: took care of a few board review tasks
Parts:
- added R211, R212: 100k, Resistors_SMD:R_0402, symbol R
Connections:
- net AVCC: no longer U202.8 (V+)
- net GNDA: now also R211.2, R212.2; no longer U202.4 (V-), U203.4 (V-)
- net VREF1_EN: now also R211.1
- net VREF2_EN: now also R212.1
- net VS_BIAS: no longer U203.11 (V+)

Commit message: reviewed footprints
they were all more or less correct, but i massaged a couple to closer match Maxim's recommended land patterns
Parts:
- U201: footprint Housings_DFN_QFN:QFN-28-1EP_4x4mm_Pitch0.4mm -> project:Maxim_90-0035
- U204, U205: footprint TO_SOT_Packages_SMD:SOT-23-6 -> project:Maxim_90-0175
Changed lines of the file:
@@
 F 0 "U201" H 8350 2400 50  0000 C CNN
 F 1 "MAX14661" H 8350 2600 50  0000 C CNN
-F 2 "Housings_DFN_QFN:QFN-28-1EP_4x4mm_Pitch0.4mm" H 8350 2500 50  0001 C CNN
+F 2 "project:Maxim_90-0035" H 8350 2500 50  0001 C CNN
 F 3 "Beyond-the-rail 16:2 multiplexer" H 8350 2300 50  0001 C CNN
 	1    8350 2500
@@
 F 0 "U205" H 5450 4650 60  0000 C CNN
 F 1 "MAX6070" H 4950 4650 60  0000 C CNN
-F 2 "TO_SOT_Packages_SMD:SOT-23-6" H 5200 4400 60  0001 C CNN
+F 2 "project:Maxim_90-0175" H 5200 4400 60  0001 C CNN
 F 3 "" H 5200 4400 60  0000 C CNN
 	1    5200 4300
@@
 F 0 "U204" H 2450 4650 60  0000 C CNN
 F 1 "MAX6070" H 1950 4650 60  0000 C CNN
-F 2 "TO_SOT_Packages_SMD:SOT-23-6" H 2200 4400 60  0001 C CNN
+F 2 "project:Maxim_90-0175" H 2200 4400 60  0001 C CNN
 F 3 "" H 2200 4400 60  0000 C CNN
 	1    2200 4300

Commit message: some notes and minor fiddling around
Parts:
- R201, R202: value R -> 0.01%
Changed lines of the file:
@@
 P 3700 6550
 F 0 "R201" V 3780 6550 50  0000 C CNN
-F 1 "R" V 3700 6550 50  0000 C CNN
+F 1 "0.01%" V 3850 6550 50  0000 C CNN
 F 2 "Resistors_SMD:R_0603" V 3630 6550 50  0001 C CNN
 F 3 "" H 3700 6550 50  0000 C CNN
@@
 P 6700 6550
 F 0 "R202" V 6780 6550 50  0000 C CNN
-F 1 "R" V 6700 6550 50  0000 C CNN
+F 1 "0.01%" V 6850 6550 50  0000 C CNN
 F 2 "Resistors_SMD:R_0603" V 6630 6550 50  0001 C CNN
 F 3 "" H 6700 6550 50  0000 C CNN
