File: thermistor-measurement-board/adc.sch (KiCad schematic (older format))
At the start: 25 parts, among them U304 MCP3911A0-E/ML, X1 ≤ 20Mz

Commit message: a few minor tweaks to thermistor board
Parts:
- added R501, R502: 0, Resistors_SMD:R_0603, symbol R
Connections:
- net OUT_A+: now also R501.1; no longer C323.2, U304.1 (CH0+)
- net OUT_A-: now also R502.1; no longer C323.1, U304.2 (CH0-)
- new net: C323.2, R501.2, U304.1 (CH0+)
- new net: C323.1, R502.2, U304.2 (CH0-)
Other:
- moved on the sheet: C324, R325, R326
Changed lines of the file:
@@
 	-1   0    0    1
 $EndComp
-Text Label 8400 2400 3    60   ~ 0
+Text Label 8600 2400 3    60   ~ 0
 OUT_B+
 $Comp
@@
 L CP1_Small C324
 U 1 1 56C03A1F
-P 8600 3200
-F 0 "C324" V 8500 3150 50  0000 L CNN
-F 1 "100p" V 8700 3100 50  0000 L CNN
-F 2 "Capacitors_SMD:C_0402" H 8600 3200 50  0001 C CNN
-F 3 "" H 8600 3200 50  0000 C CNN
-F 4 "DNP" V 8450 3200 60  0000 C CNN "Note"
-	1    8600 3200
+P 8800 3200
+F 0 "C324" V 8700 3150 50  0000 L CNN
+F 1 "100p" V 8900 3100 50  0000 L CNN
+F 2 "Capacitors_SMD:C_0402" H 8800 3200 50  0001 C CNN
+F 3 "" H 8800 3200 50  0000 C CNN
+F 4 "DNP" V 8650 3200 60  0000 C CNN "Note"
+	1    8800 3200
 	0    1    1    0
 $EndComp
-Text Label 8800 2400 3    60   ~ 0
+Text Label 9000 2400 3    60   ~ 0
 OUT_B-
 $Comp
 L R R325
 U 1 1 56C03A27
-P 8400 2950
-F 0 "R325" V 8480 2950 50  0000 C CNN
-F 1 "0" V 8400 2950 50  0000 C CNN
-F 2 "Resistors_SMD:R_0603" V 8330 2950 50  0001 C CNN
-F 3 "" H 8400 2950 50  0000 C CNN
-	1    8400 2950
+P 8600 2950
+F 0 "R325" V 8680 2950 50  0000 C CNN
+F 1 "0" V 8600 2950 50  0000 C CNN
+F 2 "Resistors_SMD:R_0603" V 8530 2950 50  0001 C CNN
+F 3 "" H 8600 2950 50  0000 C CNN
+	1    8600 2950
 	1    0    0    -1
 $EndComp
@@
 L R R326
 U 1 1 56C03A2E
-P 8800 2950
-F 0 "R326" V 8880 2950 50  0000 C CNN
-F 1 "0" V 8800 2950 50  0000 C CNN
-F 2 "Resistors_SMD:R_0603" V 8730 2950 50  0001 C CNN
-F 3 "" H 8800 2950 50  0000 C CNN
-	1    8800 2950
+P 9000 2950
+F 0 "R326" V 9080 2950 50  0000 C CNN
+F 1 "0" V 9000 2950 50  0000 C CNN
+F 2 "Resistors_SMD:R_0603" V 8930 2950 50  0001 C CNN
+F 3 "" H 9000 2950 50  0000 C CNN
+	1    9000 2950
 	1    0    0    -1
 $EndComp
@@
 	7600 4100 7500 4100
 Wire Wire Line
-	7900 2400 7900 3300
-Wire Wire Line
-	8300 2400 8300 3400
-Wire Wire Line
-	8400 3100 8400 3500
-Wire Wire Line
-	8800 3100 8800 3600
+	8600 3100 8600 3500
+Wire Wire Line
+	9000 3100 9000 3600
 Wire Wire Line
 	8000 3200 7900 3200
@@
 Connection ~ 8300 3200
 Wire Wire Line
-	8400 3200 8500 3200
-Connection ~ 8400 3200
-Wire Wire Line
-	8800 3200 8700 3200
-Connection ~ 8800 3200
-Wire Wire Line
-	8800 3600 7400 3600
-Wire Wire Line
-	8400 3500 7400 3500
-Wire Wire Line
-	8800 2800 8800 2400
-Wire Wire Line
-	8400 2400 8400 2800
+	8600 3200 8700 3200
+Connection ~ 8600 3200
+Wire Wire Line
+	9000 3200 8900 3200
+Connection ~ 9000 3200
+Wire Wire Line
+	9000 3600 7400 3600
+Wire Wire Line
+	8600 3500 7400 3500
+Wire Wire Line
+	9000 2800 9000 2400
+Wire Wire Line
+	8600 2400 8600 2800
 Text HLabel 1100 600  0    60   Input ~ 0
 DVDD
@@
 Text Notes 850  3800 0    60   ~ 0
 I/O pull resistors
+$Comp
+L R R501
+U 1 1 56C6B793
+P 7900 2950
+F 0 "R501" V 7980 2950 50  0000 C CNN
+F 1 "0" V 7900 2950 50  0000 C CNN
+F 2 "Resistors_SMD:R_0603" V 7830 2950 50  0001 C CNN
+F 3 "" H 7900 2950 50  0000 C CNN
+	1    7900 2950
+	1    0    0    -1
+$EndComp
+$Comp
+L R R502
+U 1 1 56C6B813
+P 8300 2950
+F 0 "R502" V 8380 2950 50  0000 C CNN
+F 1 "0" V 8300 2950 50  0000 C CNN
+F 2 "Resistors_SMD:R_0603" V 8230 2950 50  0001 C CNN
+F 3 "" H 8300 2950 50  0000 C CNN
+	1    8300 2950
+	1    0    0    -1
+$EndComp
+Wire Wire Line
+	7900 3100 7900 3300
+Wire Wire Line
+	8300 3100 8300 3400
+Wire Wire Line
+	7900 2400 7900 2800
+Wire Wire Line
+	8300 2800 8300 2400
 $EndSCHEMATC
